File: Console.sch (KiCad schematic (older format))
At the start: 57 parts, among them J1 batt_in, J11 lcd_out, J14 gnd_out, J17 node_conn_1, J18 node_conn_2, J2 3v3_gnd, J3 motor_out, J4 ir_out, J5 pwr_jumper, J6 gpio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

Commit message: Add Busy LED
Changed the DEF_LED to BSY_LED to indicate network business. The default led in the breakout board remains the same.
Connections:
- net DEF_LED: no longer NMCU1.D3 (GPIO0), R1.2
- new net BSY_LED: NMCU1.D3 (GPIO0), R1.2
Changed lines of the file:
@@
 $EndComp
 Text Label 5500 6200 0    50   ~ 0
-DEF_LED
+BSY_LED
 Text Label 850  2850 2    50   ~ 0
-DEF_LED
+BSY_LED
 Wire Wire Line
 	850  2850 950  2850

Commit message: Changed Switch footprint
Changed the switch to SPDT and its footprint to a mouser available switch and made all the legends visible. Added a testpoint for gnd. Final Check yet to be done
Parts:
- added TP2: TestPoint, TestPoint:TestPoint_Pad_1.5x1.5mm, symbol Connector:TestPoint
- SW1: value SW_SPST -> SW_SPDT; footprint Button_Switch_SMD:SW_DIP_SPSTx01_Slide_9.78x4.72mm_W8.61mm_P2.54mm -> Button_Switch_THT:SW_CuK_OS102011MA1QN1_SPDT_Angled; symbol Switch:SW_SPST -> Switch:SW_SPDT
Connections:
- net GND: now also TP2.1
- net SWITCH_IN: now also SW1.2 (B); no longer SW1.1 (A)
- net at J5.1 (Pin_1): now also SW1.3 (C); no longer SW1.2 (B)
Changed lines of the file:
@@
 Connection ~ 2300 4700
 Wire Wire Line
-	1900 4950 1900 4700
+	1900 4950 1900 4900
 Wire Wire Line
 	1900 4700 1750 4700
@@
 Connection ~ 1850 3000
 $Comp
-L Switch:SW_SPST SW1
+L Switch:SW_SPDT SW1
 U 1 1 5D4F2094
 P 1850 1200
 F 0 "SW1" H 1850 1435 50  0000 C CNN
-F 1 "SW_SPST" H 1850 1344 50  0000 C CNN
-F 2 "Button_Switch_SMD:SW_DIP_SPSTx01_Slide_9.78x4.72mm_W8.61mm_P2.54mm" H 1850 1200 50  0001 C CNN
+F 1 "SW_SPDT" H 1850 1344 50  0000 C CNN
+F 2 "Button_Switch_THT:SW_CuK_OS102011MA1QN1_SPDT_Angled" H 1850 1200 50  0001 C CNN
 F 3 "~" H 1850 1200 50  0001 C CNN
 	1    1850 1200
@@
 Text Notes 600  1150 0    50   ~ 0
 batt_in\n6V-12V
-Text Notes 1650 1350 0    50   ~ 0
+Text Notes 1200 1350 0    50   ~ 0
 power_switch
 Text Notes 1992 3876 0    50   ~ 0
@@
 Wire Wire Line
 	2200 1100 2200 1050
+$Comp
+L Connector:TestPoint TP2
+U 1 1 5CE2D6B9
+P 1450 5100
+F 0 "TP2" H 1508 5218 50  0000 L CNN
+F 1 "TestPoint" V 1508 5127 50  0000 L CNN
+F 2 "TestPoint:TestPoint_Pad_1.5x1.5mm" H 1650 5100 50  0001 C CNN
+F 3 "~" H 1650 5100 50  0001 C CNN
+	1    1450 5100
+	0    -1   -1   0
+$EndComp
+Wire Wire Line
+	1450 5100 1450 4900
+Wire Wire Line
+	1450 4900 1900 4900
+Connection ~ 1900 4900
+Wire Wire Line
+	1900 4900 1900 4700
+Wire Wire Line
+	2050 1200 2050 1300
 $EndSCHEMATC

Commit message: Design approved for production
Other:
- note added: "power_supply"
- note removed: "voltage_regulation"
Changed lines of the file:
@@
 	450  450  450  7850
 Text Notes 2200 550  0    50   ~ 0
-voltage_regulation
+power_supply
 Wire Wire Line
 	5500 1650 5500 1250

Commit message: Change NodeMCU Vin
Update the nodeMcu supply voltage to 5v from 3v3
Connections:
- net +3V3: no longer J17.1 (Pin_1), NMCU1.VIN
- net +5V: now also J17.1 (Pin_1), NMCU1.VIN
Changed lines of the file:
@@
 Connection ~ 3450 3000
-$Comp
-L power:+3V3 #PWR021
-U 1 1 5CCB7400
-P 5150 6050
-F 0 "#PWR021" H 5150 5900 50  0001 C CNN
-F 1 "+3V3" H 5165 6223 50  0000 C CNN
-F 2 "" H 5150 6050 50  0001 C CNN
-F 3 "" H 5150 6050 50  0001 C CNN
-	1    5150 6050
-	0    1    1    0
-$EndComp
 $Comp
 L power:+3V3 #PWR030
@@
 Wire Wire Line
 	2050 1200 2050 1300
+$Comp
+L power:+5V #PWR0101
+U 1 1 5D503C7C
+P 5150 6050
+F 0 "#PWR0101" H 5150 5900 50  0001 C CNN
+F 1 "+5V" H 5165 6223 50  0000 C CNN
+F 2 "" H 5150 6050 50  0001 C CNN
+F 3 "" H 5150 6050 50  0001 C CNN
+	1    5150 6050
+	0    1    1    0
+$EndComp
 $EndSCHEMATC
